File: hardware/Geedo_PCB_v4.kicad_sch (KiCad schematic)
At the start: 25 parts, among them J1 USB-C, J2 BATTERY, J3 OLED, SW1 MAIN_BTN, SW2 BOOT_BTN, SW3 RESET_BTN, U1 MCP73831, U2 MCP1826S-3302, U3 ESP32-C3-MINI-1

Commit message: board rev 4.3: Geedo knows his own battery
Four 0402s on the machine side. R10/R11 form a 100k/100k divider from VBAT
to IO0 (ADC1_CH0, 21 uA constant drain - years, not days), C8 filters the
midpoint, and R9 runs 10k in series from the MCP73831's STAT pin to IO1.
STAT is tri-state (LOW charging / HIGH done / Hi-Z unpowered); INPUT_PULLUP
makes Hi-Z read HIGH so LOW means exactly 'charging now'. Deliberately NOT
on IO2/IO8 - those are C3 boot-strapping pins whose pull-ups are
load-bearing, and STAT holding one low at reset would brick boot whenever
USB was plugged in.

Placement audit now checks existing copper, not just courtyards - the first
spots put R10 directly on the charger's PROG trace, caught when the router
could not escape the pad. C8's ground landed on a pour scrap fenced off by
the new tracks (no legal via site), tied to the plane with a routed stitch.

Schematic mirrors it all: IO0/IO1 pins added to the ESP32C3 symbol, parts,
power symbols and labels - with an on-wire collision guard after the first
attempt dropped a pin point onto the sheet's GND bus at y=77.47 and the
netlist checker caught CHG_STAT fused to GND. sch<->pcb: CONSISTENT.

Firmware: pollPower() plays the charging animation on USB plug-in and the
low-battery animation below 3.45 V (rate-limited, never while charging).
Boards without the divider disable sensing after three implausible reads,
so rev 4.2 and the devkit keep the old behaviour. Pure decision function,
host-tested including rollover, glitches and the no-hardware lockout.

Gates: clearance 0 (1553 items), edge 0, keepout 0, courtyards 0,
hole-to-hole 0 (85), nets split 0, GND one pour, every GND pad poured.
fab/bom.csv + cpl.csv regenerated: 19 line items, 29 placements
(100k = LCSC C25741). Anyone who exported Gerbers before this must
re-export.

Co-Authored-By: Claude Opus 5 <noreply@anthropic.com>
Claude-Session: https://claude.ai/code/session_011AnT632DFTLYxaJBrifUnG
Parts:
- added C8: 100nF, Capacitor_SMD:C_0402_1005Metric, symbol Device:C
- added R10, R11: 100k, Resistor_SMD:R_0402_1005Metric, symbol Device:R
- added R9: 10k, Resistor_SMD:R_0402_1005Metric, symbol Device:R
Connections:
- net GND: now also C8.2, R11.2
- net VBAT: now also R10.1
- net STAT_RAW: now reaches R7.1, U1.1 (STAT)
- net STAT_RAW: now also R9.1
- new net CHG_STAT: R9.2, U3.13 (IO1)
- new net VBAT_SENSE: C8.1, R10.2, R11.1, U3.12 (IO0)
